File: PLC4UNIT/(PLC4uni)/(PLC4uni).kicad_sch (KiCad schematic)
At the start: 0 parts

Commit message: USB
Other:
- removed sheet USB-Type.C
- added sheet Av (4-20) (Av 4-20(IN).kicad_sch)
- added sheet RLY_OUT_1 (RLY1.kicad_sch)
- added sheet RLY_OUT_2 (RLY1.kicad_sch)
- added sheet USB-type c (USB.kicad_sch)
- added sheet mA (4-20) (mA 4-20(IN).kicad_sch)
- sheet Av (0-10) ports: added AV_ADC, AV_IN; removed none
- sheet IN-NPN1 ports: added NPN_I1, NPN_MCU_1; removed none
- sheet IN-NPN2 ports: added NPN_I1, NPN_MCU_1; removed none
- sheet IN-NPN3 ports: added NPN_I1, NPN_MCU_1; removed none
- sheet IN-NPN4 ports: added NPN_I1, NPN_MCU_1; removed none
- sheet IN-PNP1 ports: added PNP_I1, PNP_MCU_1; removed none
- sheet IN-PNP2 ports: added PNP_I1, PNP_MCU_1; removed none
- sheet IN-PNP3 ports: added PNP_I1, PNP_MCU_1; removed none
- sheet IN-PNP4 ports: added PNP_I1, PNP_MCU_1; removed none
- sheet OUT-NPN1 ports: added NPN_MCO_1, NPN_OUT_1; removed none
- sheet OUT-NPN2 ports: added NPN_MCO_1, NPN_OUT_1; removed none
- sheet OUT-NPN3 ports: added NPN_MCO_1, NPN_OUT_1; removed none
- sheet OUT-PNP1 ports: added PNP_MCO_1, PNP_OUT_1; removed none
- sheet OUT-PNP2 ports: added PNP_MCO_1, PNP_OUT_1; removed none
- sheet OUT-PNP3 ports: added PNP_MCO_1, PNP_OUT_1; removed none
- sheet PLC4unit ports: added AV_ADC, D-minus, D-plus, RLO1, RLO2, SCLK, SDA, SEL; removed none
- sheet Power_Suply ports: added 5vusb; removed none
- sheet RS-control ports: added Con, Din, Dout, RS485-A, RS485-B; removed none
- sheet mA (0-10) ports: added Out_0-10V, SCL, SDA; removed none
- sheet mA_INTERFAZ_OUT ports: added SCLK, SDA; removed none
- note added: "IN"
- note added: "OUT"
- note removed: "ENTRADAS"
- note removed: "SALIDAS"
