File: PLC4UNIT/(PLC4uni)/Av 4-20(IN).kicad_sch (KiCad schematic)
At the start: 4 parts

Commit message: USB
Parts:
- renumbered C10 to C9, D13 to D5, R23 to R22, R25 to R24
Changed lines of the file:
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@@
 		(dnp no)
 		(fields_autoplaced yes)
-		(property "Reference" "R23"
+		(property "Reference" "R22"
 			(at 130.81 101.5999 0)
 			(effects
@@
 		(instances
 			(project "(PLC4uni)"
-				(path "/51ba3ded-ff5f-4081-8ec7-5485260143c5/2a2f8680-bcd1-449d-9473-274db87076f5"
-					(reference "R23")
+				(path "/51ba3ded-ff5f-4081-8ec7-5485260143c5/901f14ff-007b-4496-b456-fb07dd7c1be1"
+					(reference "R22")
 					(unit 1)
 				)
@@
 		(dnp no)
 		(fields_autoplaced yes)
-		(property "Reference" "#PWR061"
+		(property "Reference" "#PWR060"
 			(at 128.27 127 0)
 			(effects
@@
 		(instances
 			(project "(PLC4uni)"
-				(path "/51ba3ded-ff5f-4081-8ec7-5485260143c5/2a2f8680-bcd1-449d-9473-274db87076f5"
-					(reference "#PWR061")
+				(path "/51ba3ded-ff5f-4081-8ec7-5485260143c5/901f14ff-007b-4496-b456-fb07dd7c1be1"
+					(reference "#PWR060")
 					(unit 1)
 				)
@@
 		(dnp no)
 		(fields_autoplaced yes)
-		(property "Reference" "D13"
+		(property "Reference" "D5"
 			(at 153.67 111.7599 90)
 			(effects
@@
 		(instances
 			(project "(PLC4uni)"
-				(path "/51ba3ded-ff5f-4081-8ec7-5485260143c5/2a2f8680-bcd1-449d-9473-274db87076f5"
-					(reference "D13")
+				(path "/51ba3ded-ff5f-4081-8ec7-5485260143c5/901f14ff-007b-4496-b456-fb07dd7c1be1"
+					(reference "D5")
 					(unit 1)
 				)
@@
 		(dnp no)
 		(fields_autoplaced yes)
-		(property "Reference" "C10"
+		(property "Reference" "C9"
 			(at 142.24 113.0299 0)
 			(effects
@@
 		(instances
 			(project "(PLC4uni)"
-				(path "/51ba3ded-ff5f-4081-8ec7-5485260143c5/2a2f8680-bcd1-449d-9473-274db87076f5"
-					(reference "C10")
+				(path "/51ba3ded-ff5f-4081-8ec7-5485260143c5/901f14ff-007b-4496-b456-fb07dd7c1be1"
+					(reference "C9")
 					(unit 1)
 				)
@@
 		(dnp no)
 		(fields_autoplaced yes)
-		(property "Reference" "R25"
+		(property "Reference" "R24"
 			(at 130.81 113.0299 0)
 			(effects
@@
 		(instances
 			(project "(PLC4uni)"
-				(path "/51ba3ded-ff5f-4081-8ec7-5485260143c5/2a2f8680-bcd1-449d-9473-274db87076f5"
-					(reference "R25")
-					(unit 1)
-				)
+				(path "/51ba3ded-ff5f-4081-8ec7-5485260143c5/901f14ff-007b-4496-b456-fb07dd7c1be1"
+					(reference "R24")
+					(unit 1)
+				)
