File: PLC4UNIT/(PLC4uni)/RS-control.kicad_sch (KiCad schematic)
At the start: 1 part

Commit message: USB
Changed lines of the file:
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@@
+		)
+	)
+	(hierarchical_label "Din"
+		(shape input)
+		(at 72.39 104.14 0)
+		(effects
+			(font
+				(size 1.27 1.27)
+				(thickness 0.254)
+				(bold yes)
+			)
+			(justify left)
+		)
+	)
+	(hierarchical_label "Con"
+		(shape input)
+		(at 73.66 113.03 0)
+		(effects
+			(font
+				(size 1.27 1.27)
+				(thickness 0.254)
+				(bold yes)
+			)
+			(justify left)
 		)
 	)
@@
 		(effects
 			(font
+				(size 1.27 1.27)
+				(thickness 0.254)
+				(bold yes)
+			)
+			(justify left)
+		)
+	)
+	(hierarchical_label "Dout"
+		(shape output)
+		(at 72.39 96.52 0)
+		(effects
+			(font
